File: mainboards/L2-MB-IOP/l2-mb-iop-standart/l2-mb-iop-standart.kicad_sch (KiCad schematic)
At the start: 23 parts, among them J1 URP_Conn_01x12_Socket, J10 GPP_Conn_01x12_Socket, J11 GPP_Conn_01x12_Socket, J12 GPP_Conn_01x12_Socket, J13 GPP_Conn_01x12_Socket, J14 GPP_Conn_01x12_Socket, J15 AIP_Conn_01x12_Socket, J16 AIP_Conn_01x12_Socket, J17 AIP_Conn_01x12_Socket, J18 AIP_Conn_01x12_Socket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

Commit message: Added DCDC to L2-MB-IOP as an option so it can be used stanalone without L0 and L1.
Parts:
- added C1, C3: C, symbol Device:C
- added C2, C4: C_Polarized, symbol Device:C_Polarized
- added J23: Wire terminal_01x03_Pin, symbol Connector:Conn_01x03_Pin
- added J24: Jumper for Conn GNDs, symbol Connector:Conn_01x02_Pin
- added PS1: B240XS-1W, tuxmio:B240XS-1W, symbol tuxmio:B240XS-1W
- added PS2: B240XS-2W, tuxmio:B240XS-2W, symbol tuxmio:B240XS-2W
- added U1: LM2596s_module, tuxmio:LM2596s_module, symbol tuxmio:LM2596s_module
- added U2: LM2596_mini_module, tuxmio:LM2596_mini_module, symbol tuxmio:LM2596_mini_module
Connections:
- new net +24V: C1.1, C2.1, J23.1 (Pin_1), PS1.2 (Vi+), PS2.1 (Vi+), U1.1 (Vi-), U2.1 (Vi-)
- new net +5V: C3.1, C4.1, PS1.4 (Vo+), PS2.6 (Vo+), U1.3 (Vo-), U2.3 (Vo-)
- new net Earth: J23.3 (Pin_3)
- new net GND: C1.2, C2.2, J23.2 (Pin_2), J24.2 (Pin_2), PS1.1 (Vi-), PS2.2 (Vi-), U1.2 (Vi+), U1.4 (Vo+), U2.2 (Vi+), U2.4 (Vo+)
- new net GND1: C3.2, C4.2, J24.1 (Pin_1), PS1.3 (Vo-), PS2.4 (Vo-)
Other:
- note added: "note for future Mega 2560 has 54 digital input/output pins, of which 14 can be used for PWM output. + It also has 16 analog input pins in addition."
