File: mainboards/L2-MB-IOP/l2-mb-iop-standart/_autosave-l2-mb-iop-standart.kicad_sch (KiCad schematic)
At the start: 46 parts, among them J1 URP_Conn_01x12_Socket, J10 GPP_Conn_01x12_Socket, J11 GPP_Conn_01x12_Socket, J12 GPP_Conn_01x12_Socket, J13 GPP_Conn_01x12_Socket, J14 GPP_Conn_01x12_Socket, J15 AIP_Conn_01x12_Socket, J16 AIP_Conn_01x12_Socket, J17 AIP_Conn_01x12_Socket, J18 AIP_Conn_01x12_Socket, J19 ICP_Conn_01x12_Socket, J2 URP_Conn_01x12_Socket, J20 ICP_Conn_01x12_Socket, J21 AIP_Conn_01x12_Socket, J22 AIP_Conn_01x12_Socket, J23 Conn_01x03_Pin, J24 Conn_01x02_Pin, J25 Conn_01x02_Pin, J26 Conn_01x02_Pin, J27 Conn_01x03_Pin, J28 Conn_01x02_Pin, J29 Conn_01x02_Pin, J3 GPP_Conn_01x12_Socket, J4 GPP_Conn_01x12_Socket, J5 GPP_Conn_01x12_Socket, J6 GPP_Conn_01x12_Socket, J7 GPP_Conn_01x12_Socket, J8 GPP_Conn_01x12_Socket, J9 GPP_Conn_01x12_Socket, SW1 SW_SPDT, U1 LM2596s_module, U2 LM2596_mini_module

Commit message: Started routing L2-MB pcb.
Parts:
- gave numbers to parts that had none: 10
Changed lines of the file:
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@@
 		(dnp no)
 		(fields_autoplaced yes)
-		(property "Reference" "C?"
+		(property "Reference" "C6"
 			(at 97.79 42.2909 0)
 			(effects
@@
 			(project "l2-mb-iop-standart"
 				(path "/f25cfa12-e490-4a92-ab8c-1b3ce123d4e0"
-					(reference "C?")
+					(reference "C6")
 					(unit 1)
 				)
@@
 		(dnp no)
 		(fields_autoplaced yes)
-		(property "Reference" "C?"
+		(property "Reference" "C5"
 			(at 86.36 42.2909 0)
 			(effects
@@
 			(project ""
 				(path "/f25cfa12-e490-4a92-ab8c-1b3ce123d4e0"
-					(reference "C?")
+					(reference "C5")
 					(unit 1)
 				)
@@
 		(dnp no)
 		(fields_autoplaced yes)
-		(property "Reference" "D?"
+		(property "Reference" "D2"
 			(at 48.5775 35.56 0)
 			(effects
@@
 			(project ""
 				(path "/f25cfa12-e490-4a92-ab8c-1b3ce123d4e0"
-					(reference "D?")
+					(reference "D2")
 					(unit 1)
 				)
@@
 		(dnp no)
 		(fields_autoplaced yes)
-		(property "Reference" "C?"
+		(property "Reference" "C1"
 			(at 60.96 43.1799 0)
 			(effects
@@
 			(project ""
 				(path "/f25cfa12-e490-4a92-ab8c-1b3ce123d4e0"
-					(reference "C?")
+					(reference "C1")
 					(unit 1)
 				)
@@
 		(dnp no)
 		(fields_autoplaced yes)
-		(property "Reference" "C?"
+		(property "Reference" "C7"
 			(at 97.79 85.4709 0)
 			(effects
@@
 			(project ""
 				(path "/f25cfa12-e490-4a92-ab8c-1b3ce123d4e0"
-					(reference "C?")
+					(reference "C7")
 					(unit 1)
 				)
@@
 		(dnp no)
 		(fields_autoplaced yes)
-		(property "Reference" "D?"
+		(property "Reference" "D1"
 			(at 48.5775 26.67 0)
 			(effects
@@
 			(project "l2-mb-iop-standart"
 				(path "/f25cfa12-e490-4a92-ab8c-1b3ce123d4e0"
-					(reference "D?")
+					(reference "D1")
 					(unit 1)
 				)
@@
 		(dnp no)
 		(fields_autoplaced yes)
-		(property "Reference" "C?"
+		(property "Reference" "C8"
 			(at 110.49 85.4709 0)
 			(effects
@@
 			(project "l2-mb-iop-standart"
 				(path "/f25cfa12-e490-4a92-ab8c-1b3ce123d4e0"
-					(reference "C?")
+					(reference "C8")
 					(unit 1)
 				)
@@
 		(dnp no)
 		(fields_autoplaced yes)
-		(property "Reference" "C?"
+		(property "Reference" "C4"
 			(at 85.09 86.3599 0)
 			(effects
@@
 			(project "l2-mb-iop-standart"
 				(path "/f25cfa12-e490-4a92-ab8c-1b3ce123d4e0"
-					(reference "C?")
+					(reference "C4")
 					(unit 1)
 				)
@@
 		(dnp no)
 		(fields_autoplaced yes)
-		(property "Reference" "C?"
+		(property "Reference" "C2"
 			(at 73.66 43.1799 0)
 			(effects
@@
 			(project "l2-mb-iop-standart"
 				(path "/f25cfa12-e490-4a92-ab8c-1b3ce123d4e0"
-					(reference "C?")
+					(reference "C2")
 					(unit 1)
 				)
@@
 		(dnp no)
 		(fields_autoplaced yes)
-		(property "Reference" "C?"
+		(property "Reference" "C3"
 			(at 73.66 86.3599 0)
 			(effects
@@
 			(project ""
 				(path "/f25cfa12-e490-4a92-ab8c-1b3ce123d4e0"
-					(reference "C?")
+					(reference "C3")
 					(unit 1)
 				)
