File: mainboards/L2-MB-IOP/l2-mb-iop-standart/l2-mb-iop-standart.kicad_pcb (KiCad board)
At the start: 2 copper layers, 100 x 90 mm, 43 parts, among them J1 Conn_01x03_Pin, J10 Conn_01x01_Pin, J11 Conn_01x01_Pin, J12 Conn_01x01_Pin, J13 Conn_01x01_Pin, J14 URP_Conn_01x12_Socket, J15 URP_Conn_01x12_Socket, J16 GPP_Conn_01x12_Socket, J17 GPP_Conn_01x12_Socket, J18 GPP_Conn_01x12_Socket, J19 GPP_Conn_01x12_Socket, J2 Conn_01x01_Pin, J20 GPP_Conn_01x12_Socket, J21 GPP_Conn_01x12_Socket, J22 GPP_Conn_01x12_Socket, J23 GPP_Conn_01x12_Socket, J24 GPP_Conn_01x12_Socket, J25 GPP_Conn_01x12_Socket, J26 GPP_Conn_01x12_Socket, J27 GPP_Conn_01x12_Socket, J28 AIP_Conn_01x12_Socket, J29 AIP_Conn_01x12_Socket, J3 Conn_01x01_Pin, J30 AIP_Conn_01x12_Socket, J31 AIP_Conn_01x12_Socket, J32 ICP_Conn_01x12_Socket, J33 ICP_Conn_01x12_Socket, J34 AIP_Conn_01x12_Socket, J35 AIP_Conn_01x12_Socket, J4 Conn_01x01_Pin, J5 Conn_01x01_Pin, J6 Conn_01x01_Pin, J7 Conn_01x01_Pin, J8 Conn_01x01_Pin, J9 Conn_01x01_Pin

Commit message: Made some corrections after assembling of prototype PCBs
Connections:
- J14 pad 5: /Diag_for_future -> +5V
- J14 pad 9: /Not_assigned -> /Diag_for_future
- J15 pad 5: /Diag_for_future -> +5V
- J15 pad 9: /Not_assigned -> /Diag_for_future
- J16 pad 5: /Diag_for_future -> +5V
- J16 pad 9: /Not_assigned -> /Diag_for_future
- J17 pad 5: /Diag_for_future -> +5V
- J17 pad 9: /Not_assigned -> /Diag_for_future
- J18 pad 5: /Diag_for_future -> +5V
- J18 pad 9: /Not_assigned -> /Diag_for_future
- J19 pad 5: /Diag_for_future -> +5V
- J19 pad 9: /Not_assigned -> /Diag_for_future
- J20 pad 5: /Diag_for_future -> +5V
- J20 pad 9: /Not_assigned -> /Diag_for_future
- J21 pad 5: /Diag_for_future -> +5V
- J21 pad 9: /Not_assigned -> /Diag_for_future
- J22 pad 5: /Diag_for_future -> +5V
- J22 pad 9: /Not_assigned -> /Diag_for_future
- J23 pad 5: /Diag_for_future -> +5V
- J23 pad 9: /Not_assigned -> /Diag_for_future
- J24 pad 5: /Diag_for_future -> +5V
- J24 pad 9: /Not_assigned -> /Diag_for_future
- J25 pad 5: /Diag_for_future -> +5V
- J25 pad 9: /Not_assigned -> /Diag_for_future
- J26 pad 5: /Diag_for_future -> +5V
- J26 pad 9: /Not_assigned -> /Diag_for_future
- J27 pad 5: /Diag_for_future -> +5V
- J27 pad 9: /Not_assigned -> /Diag_for_future
- J28 pad 5: /Diag_for_future -> +5V
- J28 pad 9: /Not_assigned -> /Diag_for_future
- J29 pad 5: /Diag_for_future -> +5V
- J29 pad 9: /Not_assigned -> /Diag_for_future
- J30 pad 5: /Diag_for_future -> +5V
- J30 pad 9: /Not_assigned -> /Diag_for_future
- J31 pad 5: /Diag_for_future -> +5V
- J31 pad 9: /Not_assigned -> /Diag_for_future
- J32 pad 5: /Diag_for_future -> +5V
- J32 pad 9: /Not_assigned -> /Diag_for_future
- J33 pad 5: /Diag_for_future -> +5V
- J33 pad 9: /Not_assigned -> /Diag_for_future
- J34 pad 5: /Diag_for_future -> +5V
- J34 pad 9: /Not_assigned -> /Diag_for_future
- J35 pad 5: /Diag_for_future -> +5V
- J35 pad 9: /Not_assigned -> /Diag_for_future
Routing:
- net /Not_assigned: track 259.4 -> 0.00 mm
- net +5V: track 52.3 -> 286.8 mm
- net /Diag_for_future: track 234.5 -> 259.4 mm
