File: io-boards/DI/DIO-50-U-5B/DIO-50-U-5B.kicad_sch (KiCad schematic)
At the start: 13 parts, among them J1 GPP_Conn_01x12_Pin, J2 Conn_01x03_Pin, J3 Conn_01x02_Socket, J4 Conn_01x02_Socket, U1 PC817

Commit message: Made some corrections after assembling of prototype PCBs
Parts:
- removed D2: ABS2, Diode_SMD:Diode_Bridge_Diotec_ABS, symbol Diode_Bridge:ABS2
- added D2: MB8S, Package_SO:OnSemi_751EP_SOIC-4_3.9x4.725mm_P2.54mm, symbol Diode_Bridge:MB8S
Connections:
- net at J3.1 (Pin_1), J4.1 (Pin_1): now also D2.4
- net at J2.2 (Pin_2), J3.2 (Pin_2), J4.2 (Pin_2)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: now also D2.3
- net at R1.1: now also D2.2 (-)
- net at U1.1: now also D2.1 (+)
Changed lines of the file:
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@@
+	)
+	(junction
+		(at 146.05 82.55)
+		(diameter 0)
+		(color 0 0 0 0)
 	)
 	(junction
@@
 	)
 	(junction
-		(at 146.05 113.03)
+		(at 149.86 80.01)
 		(diameter 0)
 		(color 0 0 0 0)
 	)
 	(junction
-		(at 146.05 105.41)
+		(at 146.05 113.03)
 		(diameter 0)
 		(color 0 0 0 0)
@@
 	)
 	(junction
-		(at 163.83 80.01)
-		(diameter 0)
-		(color 0 0 0 0)
-	)
-	(junction
 		(at 232.41 102.87)
 		(diameter 0)
@@
 	(wire
 		(pts
-			(xy 124.46 68.58) (xy 163.83 68.58)
-		)
-		(stroke
-			(width 0)
-			(type default)
-		)
-	)
-	(wire
-		(pts
-			(xy 163.83 68.58) (xy 163.83 80.01)
+			(xy 124.46 68.58) (xy 149.86 68.58)
+		)
+		(stroke
+			(width 0)
+			(type default)
+		)
+	)
+	(wire
+		(pts
+			(xy 149.86 68.58) (xy 149.86 80.01)
 		)
 		(stroke
@@
 	(wire
 		(pts
-			(xy 124.46 80.01) (xy 163.83 80.01)
+			(xy 124.46 80.01) (xy 149.86 80.01)
 		)
 		(stroke
@@
 	(wire
 		(pts
-			(xy 146.05 105.41) (xy 163.83 105.41)
-		)
-		(stroke
-			(width 0)
-			(type default)
-		)
-	)
-	(wire
-		(pts
 			(xy 193.04 102.87) (xy 193.04 110.49)
 		)
@@
 	(wire
 		(pts
-			(xy 163.83 80.01) (xy 163.83 90.17)
+			(xy 163.83 105.41) (xy 149.86 105.41)
 		)
 		(stroke
@@
 	(wire
 		(pts
-			(xy 146.05 105.41) (xy 146.05 82.55)
-		)
-		(stroke
-			(width 0)
-			(type default)
-		)
-	)
-	(wire
-		(pts
 			(xy 220.98 102.87) (xy 220.98 105.41)
 		)
@@
 	(wire
 		(pts
-			(xy 146.05 113.03) (xy 146.05 105.41)
+			(xy 146.05 82.55) (xy 146.05 113.03)
 		)
 		(stroke
@@
 	(wire
 		(pts
+			(xy 149.86 80.01) (xy 149.86 105.41)
+		)
+		(stroke
+			(width 0)
+			(type default)
+		)
+	)
+	(wire
+		(pts
 			(xy 156.21 127) (xy 146.05 127)
 		)
@@
 	(wire
 		(pts
+			(xy 163.83 82.55) (xy 146.05 82.55)
+		)
+		(stroke
+			(width 0)
+			(type default)
+		)
+	)
+	(wire
+		(pts
 			(xy 209.55 83.82) (xy 209.55 97.79)
 		)
@@
 		(pts
 			(xy 124.46 71.12) (xy 137.16 71.12)
+		)
+		(stroke
+			(width 0)
+			(type default)
+		)
+	)
+	(wire
+		(pts
+			(xy 163.83 90.17) (xy 163.83 82.55)
 		)
 		(stroke
@@
 	)
 	(symbol
+		(lib_id "Diode_Bridge:MB8S")
+		(at 163.83 97.79 0)
+		(unit 1)
+		(exclude_from_sim no)
+		(in_bom yes)
+		(on_board yes)
+		(dnp no)
+		(fields_autoplaced yes)
+		(property "Reference" "D2"
+			(at 172.72 91.3698 0)
+			(effects
+				(font
+					(size 1.27 1.27)
+				)
+			)
+		)
+		(property "Value" "MB8S"
+			(at 172.72 93.9098 0)
+			(effects
+				(font
+					(size 1.27 1.27)
+				)
+			)
+		)
+		(property "Footprint" "Package_SO:OnSemi_751EP_SOIC-4_3.9x4.725mm_P2.54mm"
+			(at 167.64 94.615 0)
+			(effects
+				(font
+					(size 1.27 1.27)
+				)
+				(justify left)
+				(hide yes)
+			)
+		)
+		(property "Datasheet" "https://www.onsemi.com/pdf/datasheet/mb8s-d.pdf"
+			(at 163.83 97.79 0)
+			(effects
+				(font
+					(size 1.27 1.27)
+				)
+				(hide yes)
+			)
+		)
+		(property "Description" "Bridge Rectifier, 560V Vrms, 35A Ifsm, 0.5A If(av), SOIC-4 (Onsemi CASE 751EP)"
+			(at 163.83 97.79 0)
+			(effects
+				(font
+					(size 1.27 1.27)
+				)
+				(hide yes)
+			)
+		)
+		(pin "2"
+		)
+		(pin "3"
+		)
+		(pin "4"
+		)
+		(pin "1"
+		)
+		(instances
+			(project ""
+				(path "/6b5a44bf-f4b0-4ec6-a555-889af43cb641"
+					(reference "D2")
+					(unit 1)
+				)
+			)
+		)
+	)
+	(symbol
 		(lib_id "Device:R")
 		(at 232.41 109.22 180)
@@
 					(unit 1)
 				)
-			)
-		)
-	)
-	(symbol
-		(lib_id "Diode_Bridge:ABS2")
-		(at 163.83 97.79 0)
-		(unit 1)
-		(exclude_from_sim no)
-		(in_bom yes)
-		(on_board yes)
-		(dnp no)
-		(fields_autoplaced yes)
-		(property "Reference" "D2"
-			(at 172.72 91.3698 0)
-			(effects
-				(font
-					(size 1.27 1.27)
-				)
-			)
-		)
-		(property "Value" "ABS2"
-			(at 172.72 93.9098 0)
-			(effects
-				(font
-					(size 1.27 1.27)
-				)
-			)
-		)
-		(property "Footprint" "Diode_SMD:Diode_Bridge_Diotec_ABS"
-			(at 167.64 94.615 0)
-			(effects
-				(font
-					(size 1.27 1.27)
-				)
-				(justify left)
-				(hide yes)
-			)
-		)
-		(property "Datasheet" "https://diotec.com/tl_files/diotec/files/pdf/datasheets/abs2.pdf"
-			(at 163.83 97.79 0)
-			(effects
-				(font
-					(size 1.27 1.27)
-				)
-				(hide yes)
-			)
-		)
-		(property "Description" "Miniature Glass Passivated Single-Phase Surface Mount Bridge Rectifiers, 140V Vrms, 0.8A If, ABS SMD package"
-			(at 163.83 97.79 0)
-			(effects
-				(font
-					(size 1.27 1.27)
-				)
-				(hide yes)
-			)
-		)
-		(pin "4"
-		)
-		(pin "2"
-		)
-		(pin "3"
-		)
-		(pin "1"
-		)
-		(instances
-			(project ""
-				(path "/6b5a44bf-f4b0-4ec6-a555-889af43cb641"
-					(reference "D2")
-					(unit 1)
-				)
